File: picopocket.kicad_sch (KiCad schematic)
At the start: 87 parts, among them IC1 AR1021, J1 Conn_02x40_Odd_Even, J2 Touchscreen, J3 Audio, Q1 BSS138, Q2 BSS138, U10 74LVC1G08, U11 74LVC1G34, U12 74LVC1G34, U13 74LVC32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

Commit message: Fix AR1021 footprint
Parts:
- IC1: footprint Package_SO:TSSOP-20_4.4x6.5mm_P0.65mm -> Package_SO:SSOP-20_5.3x7.2mm_P0.65mm
Changed lines of the file:
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@@
 			)
 		)
-		(property "Footprint" "Package_SO:TSSOP-20_4.4x6.5mm_P0.65mm"
+		(property "Footprint" "Package_SO:SSOP-20_5.3x7.2mm_P0.65mm"
 			(at 356.87 175.26 0)
 			(effects

Commit message: Change to 74HC238 (avalibility)
Parts:
- U14: value 74HCT238 -> 74HC238
Connections:
- net +3.3V: now also C28.1, U14.16 (VCC), U14.6 (G1)
- net +5V: no longer C28.1, U14.16 (VCC), U14.6 (G1)
Changed lines of the file:
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@@
 	)
 	(symbol
+		(lib_name "+3.3V_1")
+		(lib_id "power:+3.3V")
+		(at 311.15 168.91 0)
+		(unit 1)
+		(exclude_from_sim no)
+		(in_bom yes)
+		(on_board yes)
+		(dnp no)
+		(fields_autoplaced yes)
+		(property "Reference" "#PWR019"
+			(at 311.15 172.72 0)
+			(effects
+				(font
+					(size 1.27 1.27)
+				)
+				(hide yes)
+			)
+		)
+		(property "Value" "+3.3V"
+			(at 311.15 163.83 0)
+			(effects
+				(font
+					(size 1.27 1.27)
+				)
+			)
+		)
+		(property "Footprint" ""
+			(at 311.15 168.91 0)
+			(effects
+				(font
+					(size 1.27 1.27)
+				)
+				(hide yes)
+			)
+		)
+		(property "Datasheet" ""
+			(at 311.15 168.91 0)
+			(effects
+				(font
+					(size 1.27 1.27)
+				)
+				(hide yes)
+			)
+		)
+		(property "Description" "Power symbol creates a global label with name \"+3.3V\""
+			(at 311.15 168.91 0)
+			(effects
+				(font
+					(size 1.27 1.27)
+				)
+				(hide yes)
+			)
+		)
+		(pin "1"
+		)
+		(instances
+			(project "picopocket"
+				(path "/3b62769f-0dea-4b89-a33d-ede04977b7a1"
+					(reference "#PWR019")
+					(unit 1)
+				)
+			)
+		)
+	)
+	(symbol
 		(lib_id "power:GND")
 		(at 212.09 196.85 0)
@@
 	)
 	(symbol
-		(lib_id "power:+5V")
-		(at 292.1 166.37 0)
-		(unit 1)
-		(exclude_from_sim no)
-		(in_bom yes)
-		(on_board yes)
-		(dnp no)
-		(fields_autoplaced yes)
-		(property "Reference" "#PWR0119"
-			(at 292.1 170.18 0)
-			(effects
-				(font
-					(size 1.27 1.27)
-				)
-				(hide yes)
-			)
-		)
-		(property "Value" "+5V"
-			(at 292.1 161.29 0)
-			(effects
-				(font
-					(size 1.27 1.27)
-				)
-			)
-		)
-		(property "Footprint" ""
-			(at 292.1 166.37 0)
-			(effects
-				(font
-					(size 1.27 1.27)
-				)
-				(hide yes)
-			)
-		)
-		(property "Datasheet" ""
-			(at 292.1 166.37 0)
-			(effects
-				(font
-					(size 1.27 1.27)
-				)
-				(hide yes)
-			)
-		)
-		(property "Description" "Power symbol creates a global label with name \"+5V\""
-			(at 292.1 166.37 0)
-			(effects
-				(font
-					(size 1.27 1.27)
-				)
-				(hide yes)
-			)
-		)
-		(pin "1"
-		)
-		(instances
-			(project "picopocket"
-				(path "/3b62769f-0dea-4b89-a33d-ede04977b7a1"
-					(reference "#PWR0119")
-					(unit 1)
-				)
-			)
-		)
-	)
-	(symbol
 		(lib_id "Jumper:SolderJumper_2_Open")
 		(at 335.28 189.23 0)
@@
 	)
 	(symbol
-		(lib_id "power:+5V")
-		(at 290.83 194.31 90)
-		(unit 1)
-		(exclude_from_sim no)
-		(in_bom yes)
-		(on_board yes)
-		(dnp no)
-		(fields_autoplaced yes)
-		(property "Reference" "#PWR016"
-			(at 294.64 194.31 0)
-			(effects
-				(font
-					(size 1.27 1.27)
-				)
-				(hide yes)
-			)
-		)
-		(property "Value" "+5V"
-			(at 287.02 194.3099 90)
-			(effects
-				(font
-					(size 1.27 1.27)
-				)
-				(justify left)
-			)
-		)
-		(property "Footprint" ""
-			(at 290.83 194.31 0)
-			(effects
-				(font
-					(size 1.27 1.27)
-				)
-				(hide yes)
-			)
-		)
-		(property "Datasheet" ""
-			(at 290.83 194.31 0)
-			(effects
-				(font
-					(size 1.27 1.27)
-				)
-				(hide yes)
-			)
-		)
-		(property "Description" "Power symbol creates a global label with name \"+5V\""
-			(at 290.83 194.31 0)
-			(effects
-				(font
-					(size 1.27 1.27)
-				)
-				(hide yes)
-			)
-		)
-		(pin "1"
-		)
-		(instances
-			(project "picopocket"
-				(path "/3b62769f-0dea-4b89-a33d-ede04977b7a1"
-					(reference "#PWR016")
-					(unit 1)
-				)
-			)
-		)
-	)
-	(symbol
 		(lib_id "Jumper:SolderJumper_2_Open")
 		(at 335.28 184.15 0)
@@
 	)
 	(symbol
-		(lib_id "Diode:ESD5Zxx")
-		(at 77.47 52.07 270)
+		(lib_name "+3.3V_1")
+		(lib_id "power:+3.3V")
+		(at 290.83 194.31 90)
 		(unit 1)
 		(exclude_from_sim no)
@@
 		(dnp no)
 		(fields_autoplaced yes)
-		(property "Reference" "D3"
-			(at 80.01 50.7999 90)
+		(property "Reference" "#PWR016"
+			(at 294.64 194.31 0)
 			(effects
 				(font
 					(size 1.27 1.27)
 				)
-				(justify left)
+				(hide yes)
 			)
 		)
-		(property "Value" "ESD5Z3.3"
-			(at 80.01 53.3399 90)
+		(property "Value" "+3.3V"
+			(at 287.02 194.3099 90)
 			(effects
 				(font
@@
 			)
 		)
-		(property "Footprint" "Diode_SMD:D_SOD-523"
-			(at 73.025 52.07 0)
+		(property "Footprint" ""
+			(at 290.83 194.31 0)
 			(effects
 				(font
@@
 			)
 		)
-		(property "Datasheet" "https://www.onsemi.com/pdf/datasheet/esd5z2.5t1-d.pdf"
-			(at 77.47 52.07 0)
+		(property "Datasheet" ""
+			(at 290.83 194.31 0)
 			(effects
 				(font
@@
 			)
 		)
-		(property "Description" "ESD Protection Diode, SOD-523"
-			(at 77.47 52.07 0)
+		(property "Description" "Power symbol creates a global label with name \"+3.3V\""
+			(at 290.83 194.31 0)
 			(effects
 				(font
@@
 			)
 		)
-		(pin "2"
-		)
 		(pin "1"
 		)
@@
 			(project "picopocket"
 				(path "/3b62769f-0dea-4b89-a33d-ede04977b7a1"
-					(reference "D3")
+					(reference "#PWR016")
 					(unit 1)
 				)
@@
 	)
 	(symbol
-		(lib_id "power:+5V")
-		(at 311.15 168.91 0)
+		(lib_id "Diode:ESD5Zxx")
+		(at 77.47 52.07 270)
 		(unit 1)
 		(exclude_from_sim no)
@@
 		(dnp no)
 		(fields_autoplaced yes)
-		(property "Reference" "#PWR019"
-			(at 311.15 172.72 0)
+		(property "Reference" "D3"
+			(at 80.01 50.7999 90)
 			(effects
 				(font
 					(size 1.27 1.27)
 				)
-				(hide yes)
+				(justify left)
 			)
 		)
-		(property "Value" "+5V"
-			(at 311.15 163.83 0)
+		(property "Value" "ESD5Z3.3"
+			(at 80.01 53.3399 90)
 			(effects
 				(font
 					(size 1.27 1.27)
 				)
+				(justify left)
 			)
 		)
-		(property "Footprint" ""
-			(at 311.15 168.91 0)
+		(property "Footprint" "Diode_SMD:D_SOD-523"
+			(at 73.025 52.07 0)
 			(effects
 				(font
@@
 			)
 		)
-		(property "Datasheet" ""
-			(at 311.15 168.91 0)
+		(property "Datasheet" "https://www.onsemi.com/pdf/datasheet/esd5z2.5t1-d.pdf"
+			(at 77.47 52.07 0)
 			(effects
 				(font
@@
 			)
 		)
-		(property "Description" "Power symbol creates a global label with name \"+5V\""
-			(at 311.15 168.91 0)
+		(property "Description" "ESD Protection Diode, SOD-523"
+			(at 77.47 52.07 0)
 			(effects
 				(font
@@
 			)
 		)
+		(pin "2"
+		)
 		(pin "1"
 		)
@@
 			(project "picopocket"
 				(path "/3b62769f-0dea-4b89-a33d-ede04977b7a1"
-					(reference "#PWR019")
+					(reference "D3")
 					(unit 1)
 				)
@@
 	)
 	(symbol
+		(lib_name "+3.3V_1")
+		(lib_id "power:+3.3V")
+		(at 292.1 166.37 0)
+		(unit 1)
+		(exclude_from_sim no)
+		(in_bom yes)
+		(on_board yes)
+		(dnp no)
+		(fields_autoplaced yes)
+		(property "Reference" "#PWR0119"
+			(at 292.1 170.18 0)
+			(effects
+				(font
+					(size 1.27 1.27)
+				)
+				(hide yes)
+			)
+		)
+		(property "Value" "+3.3V"
+			(at 292.1 161.29 0)
+			(effects
+				(font
+					(size 1.27 1.27)
+				)
+			)
+		)
+		(property "Footprint" ""
+			(at 292.1 166.37 0)
+			(effects
+				(font
+					(size 1.27 1.27)
+				)
+				(hide yes)
+			)
+		)
+		(property "Datasheet" ""
+			(at 292.1 166.37 0)
+			(effects
+				(font
+					(size 1.27 1.27)
+				)
+				(hide yes)
+			)
+		)
+		(property "Description" "Power symbol creates a global label with name \"+3.3V\""
+			(at 292.1 166.37 0)
+			(effects
+				(font
+					(size 1.27 1.27)
+				)
+				(hide yes)
+			)
+		)
+		(pin "1"
+		)
+		(instances
+			(project "picopocket"
+				(path "/3b62769f-0dea-4b89-a33d-ede04977b7a1"
+					(reference "#PWR0119")
+					(unit 1)
+				)
+			)
+		)
+	)
+	(symbol
 		(lib_id "power:GND")
 		(at 273.05 152.4 0)
@@
 			)
 		)
-		(property "Value" "74HCT238"
+		(property "Value" "74HC238"
 			(at 313.3441 171.45 0)
 			(effects

Commit message: Replace to correct mounting hole, reroute accordingly
Parts:
- H1, H2, H3, H4: footprint MountingHole:MountingHole_2.2mm_M2_ISO7380 -> MountingHole:MountingHole_2.7mm_M2.5_ISO14580_Pad
Changed lines of the file:
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@@
 			)
 		)
-		(property "Footprint" "MountingHole:MountingHole_2.2mm_M2_ISO7380"
+		(property "Footprint" "MountingHole:MountingHole_2.7mm_M2.5_ISO14580_Pad"
 			(at 388.62 243.84 0)
 			(effects
@@
 			)
 		)
-		(property "Footprint" "MountingHole:MountingHole_2.2mm_M2_ISO7380"
+		(property "Footprint" "MountingHole:MountingHole_2.7mm_M2.5_ISO14580_Pad"
 			(at 388.62 224.79 0)
 			(effects
@@
 			)
 		)
-		(property "Footprint" "MountingHole:MountingHole_2.2mm_M2_ISO7380"
+		(property "Footprint" "MountingHole:MountingHole_2.7mm_M2.5_ISO14580_Pad"
 			(at 388.62 231.14 0)
 			(effects
@@
 			)
 		)
-		(property "Footprint" "MountingHole:MountingHole_2.2mm_M2_ISO7380"
+		(property "Footprint" "MountingHole:MountingHole_2.7mm_M2.5_ISO14580_Pad"
 			(at 388.62 237.49 0)
 			(effects

Commit message: Add jlcpcb part numbers
Parts:
- C1, C2: MPN (none) -> C376807
- C10, C11: MPN (none) -> C107082
- C12, C13: MPN (none) -> C444884
- C14, C15, C16, C17, C18, C19, C20, C21, C22, C23, C24, C25, C26, C27, C28: MPN (none) -> C5142565
- C3, C4, C5, C9: MPN (none) -> C361203
- C6: MPN (none) -> C1713
- C7, C8: MPN (none) -> C385032
- D1, D2, D7, D8, D9: MPN (none) -> C475685
- D3, D4, D5, D6: MPN (none) -> C475684
- FB1, FB2: MPN (none) -> C124102
- IC1: MPN (none) -> C220291
- J1, J2, J3, U1: now left out of the parts list
- Q1, Q2: MPN (none) -> C5337205
- R1, R2, R3, R4: MPN C103904 -> C163811
- R10: MPN C103904 -> C176119
- R11: MPN (none) -> C163811
- R12, R15: MPN (none) -> C176119
- R13, R14, R8, R9: MPN (none) -> C3152105
- R5: MPN (none) -> C3017501
- R6, R7: MPN (none) -> C3015779
- U10: MPN (none) -> C434068
- U11, U12: MPN (none) -> C840096
- U13: MPN (none) -> C352974
- U14: MPN (none) -> C60434
- U15: MPN (none) -> C153798
- U16: MPN (none) -> C131154
- U3, U4, U5: MPN (none) -> C6082
- U6: value APS6404L-3SQR-SN -> LY68L6400SLIT; MPN (none) -> C261881
- U7: MPN (none) -> C840103
- U8: MPN (none) -> C75069
- U9: MPN (none) -> C460517
