File: carrierboard/carrierboard.kicad_pcb (KiCad board)
At the start: 2 copper layers, 158.3 x 63.5 mm, 30 parts, among them J1 Conn_02x40_Odd_Even, J2 USB_C_Receptacle_USB2.0_16P, J3 Bus_ISA_16bit, J4 Conn_01x03, J5 AudioJack2_Ground, J6 Conn_01x03, SW1 SW_Push, SW2 SW_Push, U1 FUSB303BTMX, U2 AP2141DWG

Commit message: Prepare next rev as published V1.0 has bugs
Other:
- board text added: "Picopocket carrier V1.0.x"
- board text removed: "Picopocket carrier V1.0"
Changed lines of the file:
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@@
 		)
 	)
-	(gr_text "Picopocket carrier V1.0"
+	(gr_text "Picopocket carrier V1.0.x"
 		(at 199.25 89.9 0)
 		(layer "B.SilkS")

Commit message: Fix traces from group move
Routing:
- net GIO8: track 88.4 -> 89.8 mm
- net GIO9: track 89.7 -> 91.1 mm
- net GIO5: track 110.2 -> 108.8 mm
- net GIO4: track 98.2 -> 96.8 mm
Changed lines of the file:
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@@
 	)
 	(segment
+		(start 171.5138 118.5071)
+		(end 171.9137 118.907)
+		(width 0.2)
+		(layer "F.Cu")
+		(net 30)
+	)
+	(segment
 		(start 251.4 114.848)
 		(end 251.6 115.048)
@@
 	)
 	(segment
-		(start 210.9306 120.2383)
-		(end 229.2 138.5077)
-		(width 0.2)
-		(layer "F.Cu")
-		(net 30)
-	)
-	(segment
 		(start 164.6965 118.0071)
 		(end 164.6965 117.5243)
@@
 	)
 	(segment
-		(start 171.5138 118.5071)
-		(end 171.9137 118.907)
-		(width 0.2)
-		(layer "F.Cu")
-		(net 30)
-	)
-	(segment
 		(start 251.6 117)
 		(end 253.3 118.7)
@@
 	)
 	(segment
-		(start 172.903986 120.2383)
-		(end 210.9306 120.2383)
-		(width 0.2)
-		(layer "F.Cu")
-		(net 30)
-	)
-	(segment
 		(start 163.2763 119.9903)
 		(end 164.1786 119.088)
@@
 	)
 	(segment
-		(start 229.2 138.5077)
-		(end 229.2 140.2)
-		(width 0.2)
-		(layer "F.Cu")
-		(net 30)
-	)
-	(segment
 		(start 170.2137 118.5071)
 		(end 171.5138 118.5071)
@@
 	)
 	(segment
-		(start 171.9137 118.907)
-		(end 171.9137 119.248014)
-		(width 0.2)
+		(start 247.65 114.848)
+		(end 251.4 114.848)
+		(width 0.3)
 		(layer "F.Cu")
 		(net 30)
 	)
 	(segment
-		(start 247.65 114.848)
-		(end 251.4 114.848)
-		(width 0.3)
+		(start 229.2 138.5077)
+		(end 229.2 140.2)
+		(width 0.2)
 		(layer "F.Cu")
 		(net 30)
@@
 	)
 	(segment
+		(start 171.9137 119.248014)
+		(end 176.065686 123.4)
+		(width 0.2)
+		(layer "F.Cu")
+		(net 30)
+	)
+	(segment
 		(start 244.925 120.948)
 		(end 243.912 119.936)
@@
 	)
 	(segment
+		(start 214.0923 123.4)
+		(end 229.2 138.5077)
+		(width 0.2)
+		(layer "F.Cu")
+		(net 30)
+	)
+	(segment
 		(start 169.0172 118.0071)
 		(end 168.9136 117.9035)
@@
 	)
 	(segment
-		(start 171.9137 119.248014)
-		(end 172.903986 120.2383)
+		(start 171.9137 118.907)
+		(end 171.9137 119.248014)
+		(width 0.2)
+		(layer "F.Cu")
+		(net 30)
+	)
+	(segment
+		(start 176.065686 123.4)
+		(end 214.0923 123.4)
 		(width 0.2)
 		(layer "F.Cu")
@@
 	)
 	(segment
-		(start 248.2 113.198)
-		(end 244.6 113.198)
+		(start 244.6 113.198)
+		(end 181.902 113.198)
 		(width 0.2)
 		(layer "F.Cu")
@@
 	)
 	(segment
-		(start 172 120.7)
-		(end 171.3071 120.0071)
+		(start 248.2 113.198)
+		(end 244.6 113.198)
 		(width 0.2)
 		(layer "F.Cu")
@@
 	)
 	(segment
-		(start 179.2969 115.3462)
-		(end 173.394 115.3462)
+		(start 172 120.7)
+		(end 171.3071 120.0071)
 		(width 0.2)
 		(layer "F.Cu")
@@
 	)
 	(segment
-		(start 244.6 113.198)
-		(end 184.8431 113.198)
+		(start 181.902 113.198)
+		(end 179.7538 115.3462)
 		(width 0.2)
 		(layer "F.Cu")
@@
 	)
 	(segment
-		(start 184.8431 109.8)
-		(end 179.2969 115.3462)
+		(start 179.7538 115.3462)
+		(end 173.394 115.3462)
 		(width 0.2)
 		(layer "F.Cu")
@@
 	)
 	(segment
-		(start 173.2163 119.6163)
-		(end 211.1163 119.6163)
+		(start 214.4 122.9)
+		(end 231.7 140.2)
 		(width 0.2)
 		(layer "F.Cu")
@@
 	)
 	(segment
-		(start 171.3052 117.0071)
-		(end 172.1644 117.8663)
+		(start 172.1644 117.8663)
+		(end 172.1644 118.5644)
 		(width 0.2)
 		(layer "F.Cu")
@@
 	)
 	(segment
-		(start 211.1163 119.6163)
-		(end 231.7 140.2)
+		(start 170.2137 117.0071)
+		(end 171.3052 117.0071)
 		(width 0.2)
 		(layer "F.Cu")
@@
 	(segment
 		(start 172.1644 118.5644)
-		(end 173.2163 119.6163)
+		(end 176.5 122.9)
 		(width 0.2)
 		(layer "F.Cu")
@@
 	)
 	(segment
-		(start 172.1644 117.8663)
-		(end 172.1644 118.5644)
+		(start 171.3052 117.0071)
+		(end 172.1644 117.8663)
 		(width 0.2)
 		(layer "F.Cu")
@@
 	)
 	(segment
-		(start 170.2137 117.0071)
-		(end 171.3052 117.0071)
+		(start 176.5 122.9)
+		(end 214.4 122.9)
 		(width 0.2)
 		(layer "F.Cu")
@@
 	)
 	(segment
-		(start 251.72 124.418)
-		(end 251.67 124.468)
+		(start 249.864315 124.468)
+		(end 250.8 124.468)
 		(width 0.2)
 		(layer "F.Cu")
@@
 	)
 	(segment
-		(start 251.67 124.468)
-		(end 250.8 124.468)
+		(start 234.978768 119.078768)
+		(end 239.5 123.6)
+		(width 0.2)
+		(layer "F.Cu")
+		(net 85)
+	)
+	(segment
+		(start 173.421232 119.078768)
+		(end 173.429464 119.087)
+		(width 0.2)
+		(layer "F.Cu")
+		(net 85)
+	)
+	(segment
+		(start 251.72 124.418)
+		(end 251.67 124.468)
 		(width 0.2)
 		(layer "F.Cu")
@@
 	)
 	(segment
-		(start 247.4953 122.485)
-		(end 248.5436 123.5333)
+		(start 251.67 124.468)
+		(end 250.8 124.468)
 		(width 0.2)
 		(layer "F.Cu")
@@
 	)
 	(segment
-		(start 248.929615 123.5333)
+		(start 248.996315 123.6)
 		(end 249.864315 124.468)
 		(width 0.2)
@@
 	)
 	(segment
-		(start 172.715932 118.373468)
-		(end 173.429464 119.087)
+		(start 173.421232 119.078768)
+		(end 234.978768 119.078768)
 		(width 0.2)
 		(layer "F.Cu")
@@
 	)
 	(segment
-		(start 173.429464 122.485)
-		(end 247.4953 122.485)
+		(start 239.5 123.6)
+		(end 248.996315 123.6)
 		(width 0.2)
 		(layer "F.Cu")
@@
 	)
 	(segment
-		(start 249.864315 124.468)
-		(end 250.8 124.468)
-		(width 0.2)
-		(layer "F.Cu")
-		(net 85)
-	)
-	(segment
-		(start 248.5436 123.5333)
-		(end 248.929615 123.5333)
+		(start 172.715932 118.373468)
+		(end 173.421232 119.078768)
 		(width 0.2)
 		(layer "F.Cu")
@@
 	)
 	(segment
+		(start 173.2572 117.9768)
+		(end 173.959168 118.678768)
+		(width 0.2)
+		(layer "F.Cu")
+		(net 89)
+	)
+	(segment
+		(start 239.665686 123.2)
+		(end 249.88 123.2)
+		(width 0.2)
+		(layer "F.Cu")
+		(net 89)
+	)
+	(segment
 		(start 167.389943 117.283243)
 		(end 167.1138 117.0071)
@@
 	)
 	(segment
-		(start 249.93 123.968)
-		(end 249.88 123.918)
+		(start 249.88 123.918)
+		(end 249.88 123.2)
 		(width 0.2)
 		(layer "F.Cu")
@@
 	)
 	(segment
-		(start 173.2572 117.9768)
-		(end 173.7824 118.502)
+		(start 249.93 123.968)
+		(end 249.88 123.918)
 		(width 0.2)
 		(layer "F.Cu")
@@
 	)
 	(segment
-		(start 167.1138 117.0071)
-		(end 165.8137 117.0071)
+		(start 173.959168 118.678768)
+		(end 235.144454 118.678768)
 		(width 0.2)
 		(layer "F.Cu")
@@
 	)
 	(segment
-		(start 249.93 122.968)
-		(end 250.8 122.968)
+		(start 235.144454 118.678768)
+		(end 239.665686 123.2)
 		(width 0.2)
 		(layer "F.Cu")
@@
 	)
 	(segment
-		(start 248.0283 121.9)
-		(end 249.0963 122.968)
+		(start 167.1138 117.0071)
+		(end 165.8137 117.0071)
 		(width 0.2)
 		(layer "F.Cu")
@@
 	)
 	(segment
-		(start 249.0963 122.968)
-		(end 249.93 122.968)
+		(start 249.93 122.968)
+		(end 250.8 122.968)
 		(width 0.2)
 		(layer "F.Cu")
@@
 	)
 	(segment
-		(start 249.88 123.918)
+		(start 249.88 123.2)
 		(end 249.88 123.018)
 		(width 0.2)
@@
 		(net 89)
 	)
-	(segment
-		(start 173.7824 121.9)
-		(end 248.0283 121.9)
-		(width 0.2)
-		(layer "F.Cu")
-		(net 89)
-	)
 	(via
 		(at 173.2572 117.9768)
@@
 	)
 	(segment
-		(start 176.8141 113.3163)
-		(end 182.323 107.8074)
-		(width 0.2)
-		(layer "F.Cu")
-		(net 93)
-	)
-	(segment
-		(start 173.8421 113.3163)
-		(end 176.8141 113.3163)
+		(start 172.8913 112.5424)
+		(end 173.0682 112.5424)
 		(width 0.2)
 		(layer "F.Cu")
@@
 	)
 	(segment
-		(start 173.0682 112.5424)
-		(end 173.8421 113.3163)
-		(width 0.2)
-		(layer "F.Cu")
-		(net 93)
-	)
-	(segment
 		(start 246.3 111.398)
 		(end 244.6 109.698)
@@
 	)
 	(segment
-		(start 172.8913 112.5424)
-		(end 173.0682 112.5424)
+		(start 173.8421 113.3163)
+		(end 176.814214 113.3163)
 		(width 0.2)
 		(layer "F.Cu")
@@
 		(width 0.2)
 		(layer "F.Cu")
+		(net 93)
+	)
+	(segment
+		(start 178.925114 111.2054)
+		(end 182.323 111.2054)
+		(width 0.2)
+		(layer "F.Cu")
+		(net 93)
+	)
+	(segment
+		(start 173.0682 112.5424)
+		(end 173.8421 113.3163)
+		(width 0.2)
+		(layer "F.Cu")
+		(net 93)
+	)
+	(segment
+		(start 176.814214 113.3163)
+		(end 178.925114 111.2054)
+		(width 0.2)
+		(layer "F.Cu")
