File: companionboard/companion_board.kicad_sch (KiCad schematic)
At the start: 6 parts, among them J1 Conn_02x07_Odd_Even, J2 USB_A, J3 USB_B_Micro, J4 Conn_01x03, SW1 SW_SPDT, SW2 SW_Push

Commit message: Update companionboard with line in input
Parts:
- added C1: 10p, Capacitor_SMD:C_0805_2012Metric, symbol Device:C
- added C2: 10µ, Capacitor_SMD:C_0805_2012Metric, symbol Device:C
- added C3: 10n, Capacitor_SMD:C_0805_2012Metric, symbol Device:C
- added J5: Conn_02x07_Odd_Even, Connector_PinSocket_2.00mm:PinSocket_2x07_P2.00mm_Vertical, symbol Connector_Generic:Conn_02x07_Odd_Even
- added J6: Conn_01x03_Pin, Connector_PinHeader_2.54mm:PinHeader_1x03_P2.54mm_Vertical, symbol Connector:Conn_01x03_Pin
- added JP1: SolderJumper_3_Open, Jumper:SolderJumper-3_P2.0mm_Open_TrianglePad1.0x1.5mm, symbol Jumper:SolderJumper_3_Open
- added Q1: BC857, Package_TO_SOT_SMD:SOT-23, symbol Transistor_BJT:BC857
- added Q2: BC847, Package_TO_SOT_SMD:SOT-23, symbol Transistor_BJT:BC847
- added R1, R4: 22k, Resistor_SMD:R_0402_1005Metric_Pad0.72x0.64mm_HandSolder, symbol Device:R
- added R2, R3: 33k, Resistor_SMD:R_0402_1005Metric_Pad0.72x0.64mm_HandSolder, symbol Device:R
- added R5: 5.6k, Resistor_SMD:R_0402_1005Metric_Pad0.72x0.64mm_HandSolder, symbol Device:R
- added SW3: SW_SPDT, Button_Switch_THT:SW_Slide-03_Wuerth-WS-SLTV_10x2.5x6.4_P2.54mm, symbol Switch:SW_SPDT_312
- added U1: 74LVC1G14, Package_TO_SOT_SMD:SOT-353_SC-70-5_Handsoldering, symbol 74xGxx:74LVC1G14
- SW1: symbol Switch:SW_SPDT -> Switch:SW_SPDT_312
Connections:
- net +5V: now also SW1.3 (A), C3.1, J5.1 (Pin_1), J5.2 (Pin_2), J6.1 (Pin_1), R1.1, U1.5 (VCC); no longer SW1.1 (A)
- net BOOTSEL: now also SW1.1 (B), J5.8 (Pin_8); no longer SW1.2 (B)
- net DACK1: now also J5.6 (Pin_6)
- net DRQ1: now also J5.5 (Pin_5)
- net GIO3: now also SW3.1 (B)
- net GIO5: now also J5.9 (Pin_9)
- net GIO6: now also J5.10 (Pin_10)
- net GIO7: now also J5.11 (Pin_11)
- net GIO8: now also J5.12 (Pin_12)
- net GIO9: now also J5.13 (Pin_13)
- net GND: now also C1.2, C3.2, J5.14 (Pin_14), J5.4 (Pin_4), J6.3 (Pin_3), R4.2, U1.3 (GND); no longer J1.3 (Pin_3)
- new net: J1.3 (Pin_3), J5.3 (Pin_3), JP1.1 (A)
- new net: J5.7 (Pin_7), JP1.3 (B)
- new net: R5.1, SW3.3 (A), U1.4
- new net: Q1.2 (E), Q2.2 (E), R5.2
- new net: Q1.1 (B), R1.2, R2.1
- new net: C2.1, J6.2 (Pin_2)
- new net: C2.2, R2.2, R3.1
- new net: Q2.1 (B), R3.2, R4.1
- new net: C1.1, Q1.3 (C), Q2.3 (C), U1.2
- new net: JP1.2 (C), SW3.2 (C)
- no-connect marks 0 -> 2

Commit message: Tidy up board
Parts:
- added F1: Fuse_Small, Fuse:Fuse_0805_2012Metric, symbol Device:Fuse_Small
Connections:
- net +5V: now also F1.2; no longer J2.1 (VBUS)
- new net: F1.1, J2.1 (VBUS)
Changed lines of the file:
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@@
+	(wire
+		(pts
+			(xy 48.26 111.76) (xy 45.72 111.76)
+		)
+		(stroke
+			(width 0)
+			(type default)
+		)
+	)
+	(wire
+		(pts
+			(xy 55.88 111.76) (xy 53.34 111.76)
+		)
+		(stroke
+			(width 0)
+			(type default)
+		)
+	)
 	(wire
 		(pts
@@
 	(symbol
 		(lib_id "power:+5V")
-		(at 45.72 111.76 270)
+		(at 55.88 111.76 270)
 		(unit 1)
 		(exclude_from_sim no)
@@
 		(fields_autoplaced yes)
 		(property "Reference" "#PWR07"
-			(at 41.91 111.76 0)
+			(at 52.07 111.76 0)
 			(effects
 				(font
@@
 		)
 		(property "Value" "+5V"
-			(at 49.53 111.7599 90)
+			(at 59.69 111.7599 90)
 			(effects
 				(font
@@
 		)
 		(property "Footprint" ""
-			(at 45.72 111.76 0)
+			(at 55.88 111.76 0)
 			(effects
 				(font
@@
 		)
 		(property "Datasheet" ""
-			(at 45.72 111.76 0)
+			(at 55.88 111.76 0)
 			(effects
 				(font
@@
 		)
 		(property "Description" "Power symbol creates a global label with name \"+5V\""
-			(at 45.72 111.76 0)
+			(at 55.88 111.76 0)
 			(effects
 				(font
@@
 					(unit 1)
 				)
+			)
+		)
+	)
+	(symbol
+		(lib_id "Device:Fuse_Small")
+		(at 50.8 111.76 0)
+		(unit 1)
+		(exclude_from_sim no)
+		(in_bom yes)
+		(on_board yes)
+		(dnp no)
+		(fields_autoplaced yes)
+		(property "Reference" "F1"
+			(at 50.8 106.68 0)
+			(effects
+				(font
+					(size 1.27 1.27)
+				)
+			)
+		)
+		(property "Value" "Fuse_Small"
+			(at 50.8 109.22 0)
+			(effects
+				(font
+					(size 1.27 1.27)
+				)
+			)
+		)
+		(property "Footprint" "Fuse:Fuse_0805_2012Metric"
+			(at 50.8 111.76 0)
+			(effects
+				(font
+					(size 1.27 1.27)
+				)
+				(hide yes)
+			)
+		)
+		(property "Datasheet" "~"
+			(at 50.8 111.76 0)
+			(effects
+				(font
+					(size 1.27 1.27)
+				)
+				(hide yes)
+			)
+		)
+		(property "Description" "Fuse, small symbol"
+			(at 50.8 111.76 0)
+			(effects
+				(font
+					(size 1.27 1.27)
+				)
+				(hide yes)
+			)
+		)
+		(pin "2"
+		)
+		(pin "1"
+		)
+		(instances
+			(project ""
+				(path "/917e9518-00c4-4cd7-970b-c5b2f2945b7d"
+					(reference "F1")
+					(unit 1)
+				)
