File: companionboard/companion_board.kicad_pcb (KiCad board)
At the start: 2 copper layers, 33 x 18.5 mm, 7 parts, among them J1 Conn_02x07_Odd_Even, J2 USB_A, J3 USB_B_Micro, J4 Conn_01x03, SW1 SW_SPDT, SW2 SW_Push

Commit message: Update companionboard with line in input
Parts:
- added C1: 10p, Capacitor_SMD:C_0805_2012Metric, F.Cu at (147.3, 70.6)
- added C2: 10µ, Capacitor_SMD:C_0805_2012Metric, B.Cu at (155.0, 70.1)
- added C3: 10n, Capacitor_SMD:C_0805_2012Metric, F.Cu at (150.9, 73.0)
- added J5: Conn_02x07_Odd_Even, Connector_PinSocket_2.00mm:PinSocket_2x07_P2.00mm_Vertical, F.Cu at (117.6, 73.7)
- added J6: Conn_01x03_Pin, Connector_PinHeader_2.54mm:PinHeader_1x03_P2.54mm_Vertical, F.Cu at (157.5, 69.9)
- added JP1: SolderJumper_3_Open, Jumper:SolderJumper-3_P2.0mm_Open_TrianglePad1.0x1.5mm, B.Cu at (114.2, 70.5)
- added Q1: BC857, Package_TO_SOT_SMD:SOT-23, B.Cu at (151.5, 66.4)
- added Q2: BC847, Package_TO_SOT_SMD:SOT-23, B.Cu at (151.4, 74.2)
- added R1: 22k, Resistor_SMD:R_0402_1005Metric_Pad0.72x0.64mm_HandSolder, B.Cu at (151.2, 68.7)
- added R2: 33k, Resistor_SMD:R_0402_1005Metric_Pad0.72x0.64mm_HandSolder, B.Cu at (152.4, 69.8)
- added R3: 33k, Resistor_SMD:R_0402_1005Metric_Pad0.72x0.64mm_HandSolder, B.Cu at (152.4, 70.8)
- added R4: 22k, Resistor_SMD:R_0402_1005Metric_Pad0.72x0.64mm_HandSolder, B.Cu at (152.3, 71.8)
- added R5: 5.6k, Resistor_SMD:R_0402_1005Metric_Pad0.72x0.64mm_HandSolder, F.Cu at (154.1, 70.3)
- added SW3: SW_SPDT, Button_Switch_THT:SW_Slide-03_Wuerth-WS-SLTV_10x2.5x6.4_P2.54mm, F.Cu at (124.8, 70.6)
- added U1: 74LVC1G14, Package_TO_SOT_SMD:SOT-353_SC-70-5_Handsoldering, F.Cu at (151.0, 70.4)
- REF**: value happyface_small -> happyface_smaller; footprint logo:happyface_small -> logo:happyface_smaller; moved to F.Cu
- moved J2 26.1 mm to (161.9, 71.5)
- moved J3 24.2 mm to (154.6, 62.8), turned to 180 degrees
- moved SW2 19.1 mm to (137.9, 67.8), turned to 90 degrees
- moved SW1 11.2 mm to (131.7, 70.7), turned to -90 degrees
- moved REF** 11.2 mm to (140.1, 77.9), turned to 0 degrees
- moved J4 8.98 mm to (124.0, 62.9), turned to 90 degrees
Connections:
- J1 pad 3: GND -> Net-(J1-Pin_3)
- SW1 pad 1: +5V -> BOOTSEL
- SW1 pad 2: BOOTSEL -> unconnected-(SW1-C-Pad2)
- SW1 pad 3: unconnected-(SW1-C-Pad3) -> +5V
Routing:
- net GND: track 44.9 -> 143.6 mm, vias 0 -> 3
- net +5V: track 47.9 -> 101.3 mm, vias 0 -> 1
- net Net-(SW3-A): track 0.00 -> 37.4 mm, vias 0 -> 1
- net GIO8: track 35.4 -> 61.0 mm
- net GIO9: track 38.6 -> 57.3 mm
- net GIO3: track 0.00 -> 17.8 mm
- net GIO5: track 18.0 -> 35.3 mm
- net GIO6: track 5.34 -> 21.2 mm
- net Net-(Q1-E): track 0.00 -> 14.7 mm, vias 0 -> 1
- net BOOTSEL: track 10.4 -> 23.7 mm
- net Net-(Q1-C): track 0.00 -> 12.3 mm, vias 0 -> 1
- net DRQ1: track 0.00 -> 12.0 mm
- net Net-(JP1-C): track 0.00 -> 11.7 mm
- net DACK1: track 0.00 -> 9.78 mm
- net GIO7: track 5.93 -> 15.2 mm, vias 1 -> 0
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Other:
- board size 33 x 18.5 mm -> 50.9 x 18.5 mm

Commit message: Tidy up board
Parts:
- added F1: Fuse_Small, Fuse:Fuse_0805_2012Metric, B.Cu at (155.3, 66.3)
- R5: moved to B.Cu
- moved C3 5.69 mm to (145.3, 72.7), turned to -90 degrees
- moved R5 4.99 mm to (152.4, 75.0), turned to 180 degrees
- moved Q1 4.80 mm to (149.3, 70.6)
- moved J4 2.59 mm to (126.6, 62.8)
- moved R1 2.38 mm to (152.4, 70.7), turned to 180 degrees
- moved C1 2.20 mm to (147.4, 72.8)
- moved Q2 2.18 mm to (149.3, 74.0)
- moved R4 2.13 mm to (152.4, 73.9)
- moved C2 2.03 mm to (155.0, 72.1)
- moved R2 2.03 mm to (152.4, 71.8)
- moved R3 2.03 mm to (152.4, 72.9)
- moved U1 2.03 mm to (151.0, 72.4)
Connections:
- J2 pad 1: +5V -> Net-(J2-VBUS)
Routing:
- net +5V: track 101.3 -> 91.1 mm
- net Net-(Q1-E): track 14.7 -> 5.85 mm, vias 1 -> 0
- net Net-(J2-VBUS): track 0.00 -> 7.35 mm
- net GND: track 143.6 -> 150.9 mm
- net Net-(Q1-C): track 12.3 -> 6.17 mm
- net Net-(Q1-B): track 7.08 -> 3.05 mm
- net Net-(SW3-A): track 37.4 -> 40.0 mm, vias 1 -> 2
- net GIO7: track 15.2 -> 17.8 mm
- net GIO6: track 21.2 -> 23.0 mm
Other:
- board size 50.9 x 18.5 mm -> 59.3 x 18.5 mm

Commit message: Fix flipped connector
Parts:
- J5: moved to B.Cu
- moved J5 2.00 mm to (119.6, 73.7), turned to 0 degrees
Routing:
- net Net-(J5-Pin_7): track 4.08 -> 6.89 mm
- net GIO8: track 61.0 -> 63.6 mm
- net DACK1: track 9.78 -> 7.22 mm
- net DRQ1: track 12.0 -> 9.72 mm, vias 0 -> 1
- net Net-(J1-Pin_3): track 7.64 -> 9.78 mm
- net GIO5: track 35.3 -> 36.4 mm
- net GIO7: track 17.8 -> 17.0 mm
- net GIO6: track 23.0 -> 22.5 mm
- net GIO3: track 17.8 -> 17.3 mm
- net GIO9: vias 0 -> 1
